Commit message: Updated URDF

File: elrik_description/urdf/elrik.urdf (robot description, URDF)
Before this commit: robot elrik, 34 links, 33 joints
Links:
- removed link base_link
- removed link camera_link
- removed link head_base_link
- removed link head_depth_cam_mount_link
- removed link left_armrot_link
- removed link left_ear_link
- removed link left_elbow_link
- removed link left_forearm_link
- removed link left_forearm_pitch_link
- removed link left_forearm_roll_link
- removed link left_forearmrot_link
- removed link left_hand_link
- removed link left_shoul_base_link
- removed link left_shoul_link
- removed link left_shoul_rot_link
- removed link left_upper_arm_link
- removed link neck_pitch_link
- removed link neck_yaw_link
- removed link right_armrot_link
- removed link right_ear_link
- removed link right_elbow_link
- removed link right_forearm_link
- removed link right_forearm_pitch_link
- removed link right_forearm_roll_link
- removed link right_forearmrot_link
- removed link right_hand_link
- removed link right_shoul_base_link
- removed link right_shoul_link
- removed link right_shoul_rot_link
- removed link right_upper_arm_link
- removed link torso_link
- removed link torso_pitch_link
- removed link torso_roll_link
- removed link torso_yaw_link
- added link world
Joints:
- removed joint base2torso_yaw_joint
- removed joint head_base2left_shoul_base_joint
- removed joint head_base2neck_yaw_joint
- removed joint head_base2right_shoul_base_joint
- removed joint head_depth_cam_mount2camera_joint
- removed joint head_depth_cam_mount2left_ear_joint
- removed joint head_depth_cam_mount2right_ear_joint
- removed joint left_arm2armrot_joint
- removed joint left_armrot2elbow_joint
- removed joint left_elbow2forearm_joint
- removed joint left_forearm2forearmrot_joint
- removed joint left_forearm_pitch2forearm_roll_joint
- removed joint left_forearm_roll2hand_joint
- removed joint left_forearmrot2forearm_pitch_joint
- removed joint left_shoul2shoul_rot_joint
- removed joint left_shoul_base2shoul_joint
- removed joint left_shoul_rot2upper_arm_joint
- removed joint neck_pitch2head_depth_cam_mount_joint
- removed joint neck_yaw2pitch_joint
- removed joint right_arm2armrot_joint
- removed joint right_armrot2elbow_joint
- removed joint right_elbow2forearm_joint
- removed joint right_forearm2forearmrot_joint
- removed joint right_forearm_pitch2forearm_roll_joint
- removed joint right_forearm_roll2hand_joint
- removed joint right_forearmrot2forearm_pitch_joint
- removed joint right_shoul2shoul_rot_joint
- removed joint right_shoul_base2shoul_joint
- removed joint right_shoul_rot2upper_arm_joint
- removed joint torso2head_base_joint
- removed joint torso_pitch2roll_joint
- removed joint torso_roll2torso_joint
- removed joint torso_yaw2pitch_joint
- added joint world_joint: type fixed, parent world, child link_torso, origin xyz=0 0 0.964145 rpy=0 0 0
