Commit message: Updated URDF

File: elrik_description/urdf/phobos_generated.urdf (robot description, URDF)
Before this commit: robot elrik, 18 links, 17 joints
Links:
- added link world
- link link_head_pitch: geometry collision box size=0.05500 0.06310 0.13950; visual mesh filename=package://elrik_description/meshes/stl/head_pitch.stl scale=1.00000 1.00000 1.00000
- link link_head_roll: geometry collision box size=0.08500 0.05150 0.03370; collision box size=0.12520 0.03016 0.02662
- link link_head_yaw: geometry collision box size=0.04200 0.06300 0.06300; visual mesh filename=package://elrik_description/meshes/stl/head_yaw.stl scale=1.00000 1.00000 1.00000
- link link_left_forearm: geometry collision box size=0.08489 0.06853 0.11616; visual mesh filename=package://elrik_description/meshes/stl/left_forearm.stl scale=1.00000 1.00000 1.00000
- link link_left_hand: geometry collision box size=0.05243 0.08957 0.26082; visual mesh filename=package://elrik_description/meshes/stl/left_hand.stl scale=1.00000 1.00000 1.00000
- link link_left_shoulder: geometry collision cylinder length=0.12980 radius=0.05019; visual mesh filename=package://elrik_description/meshes/stl/left_shoulder.stl scale=1.00000 1.00000 1.00000
- link link_left_shoulder_x: geometry collision box size=0.06396 0.10018 0.17240; visual mesh filename=package://elrik_description/meshes/stl/left_shoulder_x.stl scale=1.00000 1.00000 1.00000
- link link_left_upper_arm: geometry collision box size=0.07946 0.06203 0.26602; visual mesh filename=package://elrik_description/meshes/stl/left_upper_arm.stl scale=1.00000 1.00000 1.00000
- link link_left_wrist: geometry collision box size=0.07085 0.08614 0.19550; visual mesh filename=package://elrik_description/meshes/stl/left_wrist.stl scale=1.00000 1.00000 1.00000
- link link_left_wrist_x: geometry collision box size=0.07164 0.08000 0.06454; visual mesh filename=package://elrik_description/meshes/stl/left_wrist_x.stl scale=1.00000 1.00000 1.00000
- link link_right_forearm: geometry collision box size=0.08489 0.06853 0.11616; visual mesh filename=package://elrik_description/meshes/stl/right_forearm.stl scale=1.00000 1.00000 1.00000
- link link_right_hand: geometry collision box size=0.04897 0.08957 0.26082; visual mesh filename=package://elrik_description/meshes/stl/right_hand.stl scale=1.00000 1.00000 1.00000
- link link_right_shoulder: geometry collision cylinder length=0.13522 radius=0.04602; visual mesh filename=package://elrik_description/meshes/stl/right_shoulder.stl scale=1.00000 1.00000 1.00000
- link link_right_shoulder_x: geometry collision box size=0.06396 0.10018 0.17240; visual mesh filename=package://elrik_description/meshes/stl/right_shoulder_x.stl scale=1.00000 1.00000 1.00000
- link link_right_upper_arm: geometry collision box size=0.07946 0.06203 0.26602; visual mesh filename=package://elrik_description/meshes/stl/right_upper_arm.stl scale=1.00000 1.00000 1.00000
- link link_right_wrist: geometry collision box size=0.07085 0.08614 0.19550; visual mesh filename=package://elrik_description/meshes/stl/right_wrist.stl scale=1.00000 1.00000 1.00000
- link link_right_wrist_x: geometry collision box size=0.07164 0.08000 0.06454; visual mesh filename=package://elrik_description/meshes/stl/right_wrist_x.stl scale=1.00000 1.00000 1.00000
- link link_torso: geometry collision box size=0.38548 0.07402 0.25694; visual mesh filename=package://elrik_description/meshes/stl/torso.stl scale=1.00000 1.00000 1.00000
Joints:
- removed joint link_right_shoulder_joint
- added joint joint_right_shoulder_pitch: type revolute, parent link_torso, child link_right_shoulder, origin xyz=-0.16356 -0.00077 0.19342 rpy=0.00000 0.00000 0.00000, axis -0.86603 0.00000 0.50000, limit lower=-3.14000 upper=3.14000 effort=0.00000 velocity=0.00000
- added joint world_joint: type fixed, parent world, child link_torso, origin xyz=0 0 0.964145 rpy=0 0 0
- joint joint_left_arm_yaw: axis 0.00000 0.00000 1.00000 -> 0.00000 0.00000 -1.00000
- joint joint_left_elbow_pitch: axis 0.00000 0.00000 1.00000 -> 0.00000 0.00000 -1.00000; origin xyz=0.00011 0.00027 0.23600 rpy=-3.14159 -1.57080 -3.14159 -> xyz=0.00011 0.00027 0.23600 rpy=3.14159 -1.57080 3.14159
- joint joint_left_forearm_yaw: axis 0.00000 0.00000 1.00000 -> 0.00000 0.00000 -1.00000
- joint joint_left_shoulder_pitch: axis 0.00000 0.00000 1.00000 -> 0.00000 0.00000 -1.00000
- joint joint_left_wrist_pitch: axis 0.00000 0.00000 1.00000 -> 0.00000 0.00000 -1.00000; origin xyz=-0.00110 -0.00019 0.17400 rpy=1.79848 -1.57080 1.34311 -> xyz=-0.00110 -0.00019 0.17400 rpy=1.43744 -1.57080 1.70415
- joint joint_right_shoulder_roll: axis 0.00000 0.00000 1.00000 -> 0.00000 0.00000 -1.00000
- joint joint_right_wrist_roll: axis 0.00000 0.00000 1.00000 -> 0.00000 0.00000 -1.00000

Commit message: Updated URDF - flipped robot to face towards positive y

File: elrik_description/urdf/phobos_generated.urdf (robot description, URDF)
Before this commit: robot elrik, 19 links, 18 joints
Links:
- removed link world
Joints:
- removed joint world_joint
- joint joint_head_yaw: origin xyz=-0.00012 -0.00000 0.20400 rpy=0.00000 0.00000 0.00000 -> xyz=0.00012 0.00000 0.20400 rpy=0.00000 0.00000 -3.14159
- joint joint_left_elbow_pitch: origin xyz=0.00011 0.00027 0.23600 rpy=3.14159 -1.57080 3.14159 -> xyz=0.00011 0.00027 0.23600 rpy=3.14159 -1.57080 -3.14159
- joint joint_left_shoulder_pitch: origin xyz=0.16356 -0.00077 0.19342 rpy=0.00000 1.04720 0.00000 -> xyz=-0.16356 0.00077 0.19342 rpy=-0.00000 1.04720 -3.14159
- joint joint_right_arm_yaw: origin xyz=-0.00020 -0.12745 0.01486 rpy=1.57080 -0.00000 0.00000 -> xyz=-0.00020 -0.12745 0.01486 rpy=1.57080 0.00000 0.00000
- joint joint_right_shoulder_pitch: origin xyz=-0.16356 -0.00077 0.19342 rpy=0.00000 0.00000 0.00000 -> xyz=0.16356 0.00077 0.19342 rpy=0.00000 0.00000 -3.14159
- joint joint_right_wrist_roll: origin xyz=-0.00000 0.00000 -0.00000 rpy=1.57080 1.57080 0.00000 -> xyz=0.00000 0.00000 -0.00000 rpy=1.57080 1.57080 0.00000
