Commit message: Updated URDF

File: wattson_description/urdf/phobos_generated.urdf (robot description, URDF)
Before this commit: robot Wattson, 16 links, 15 joints
Links:
- added link link_right_hand
- added link link_right_wrist_x
- link link_right_wrist: geometry collision cylinder length=0.10977 radius=0.05250; visual mesh filename=package://wattson_description/meshes/stl/Cone.stl scale=0.01903 0.01903 0.04934
Joints:
- added joint joint_right_wrist_pitch: type revolute, parent link_right_wrist, child link_right_wrist_x, origin xyz=0.00000 -0.01442 0.15088 rpy=1.43744 -1.57080 1.70415, axis 0.00000 0.00000 1.00000, limit lower=-3.14000 upper=3.14000 effort=0.00000 velocity=0.00000
- added joint joint_right_wrist_roll: type revolute, parent link_right_wrist_x, child link_right_hand, origin xyz=-0.00000 0.02290 -0.00000 rpy=1.57080 -1.57080 0.00000, axis 0.00000 0.00000 1.00000, limit lower=-3.14000 upper=3.14000 effort=0.00000 velocity=0.00000

Commit message: Updated URDF

File: wattson_description/urdf/phobos_generated.urdf (robot description, URDF)
Before this commit: robot Wattson, 18 links, 17 joints
Links:
- removed link link_right_wrist_x
- link link_right_hand: geometry visual mesh filename=package://wattson_description/meshes/stl/Cone.stl scale=0.01903 0.01903 0.04934
- link link_right_wrist: geometry collision cylinder length=0.10977 radius=0.05250; visual mesh filename=package://wattson_description/meshes/stl/right_wrist.stl scale=1.00000 1.00000 1.00000
Joints:
- removed joint joint_right_wrist_pitch
- joint joint_right_wrist_roll: origin xyz=-0.00000 0.02290 -0.00000 rpy=1.57080 -1.57080 0.00000 -> xyz=0.00000 -0.03732 0.15088 rpy=-1.57080 0.00000 3.14159; parent link_right_wrist_x -> link_right_wrist
